File: Business_Card.kicad_sch (KiCad schematic)
At the start: 0 parts

Commit message: updated schematic
Parts:
- added BT1: Battery_Cell, Coin_Battery_Holder_CR2032:Coin_Battery_Holder_CR2032, symbol Device:Battery_Cell
Connections:
- new net +3V0: BT1.1 (+)
- new net GND: BT1.2 (-)
Other:
- title: (none) -> Business Card PCB
Changed lines of the file:
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@@
 	(generator "eeschema")
 	(generator_version "9.0")
-	(paper "A4")
+	(paper "A5")
+	(title_block
+		(title "Business Card PCB")
+		(date "2025-09-25")
+	)
+	(symbol
+		(lib_id "power:+3V0")
+		(at 36.83 34.29 0)
+		(unit 1)
+		(exclude_from_sim no)
+		(in_bom yes)
+		(on_board yes)
+		(dnp no)
+		(fields_autoplaced yes)
+		(property "Reference" "#PWR01"
+			(at 36.83 38.1 0)
+			(effects
+				(font
+					(size 1.27 1.27)
+				)
+				(hide yes)
+			)
+		)
+		(property "Value" "+3V0"
+			(at 36.83 29.21 0)
+			(effects
+				(font
+					(size 1.27 1.27)
+				)
+			)
+		)
+		(property "Footprint" ""
+			(at 36.83 34.29 0)
+			(effects
+				(font
+					(size 1.27 1.27)
+				)
+				(hide yes)
+			)
+		)
+		(property "Datasheet" ""
+			(at 36.83 34.29 0)
+			(effects
+				(font
+					(size 1.27 1.27)
+				)
+				(hide yes)
+			)
+		)
+		(property "Description" "Power symbol creates a global label with name \"+3V0\""
+			(at 36.83 34.29 0)
+			(effects
+				(font
+					(size 1.27 1.27)
+				)
+				(hide yes)
+			)
+		)
+		(pin "1"
+		)
+		(instances
+			(project ""
+				(path "/81126baf-9999-480c-992f-3520723c9b7d"
+					(reference "#PWR01")
+					(unit 1)
+				)
+			)
+		)
+	)
+	(symbol
+		(lib_id "Device:Battery_Cell")
+		(at 36.83 39.37 0)
+		(unit 1)
+		(exclude_from_sim no)
+		(in_bom yes)
+		(on_board yes)
+		(dnp no)
+		(fields_autoplaced yes)
+		(property "Reference" "BT1"
+			(at 40.64 36.2584 0)
+			(effects
+				(font
+					(size 1.27 1.27)
+				)
+				(justify left)
+			)
+		)
+		(property "Value" "Battery_Cell"
+			(at 40.64 38.7984 0)
+			(effects
+				(font
+					(size 1.27 1.27)
+				)
+				(justify left)
+			)
+		)
+		(property "Footprint" "Coin_Battery_Holder_CR2032:Coin_Battery_Holder_CR2032"
+			(at 36.83 37.846 90)
+			(effects
+				(font
+					(size 1.27 1.27)
+				)
+				(hide yes)
+			)
+		)
+		(property "Datasheet" "~"
+			(at 36.83 37.846 90)
+			(effects
+				(font
+					(size 1.27 1.27)
+				)
+				(hide yes)
+			)
+		)
+		(property "Description" "Single-cell battery"
+			(at 36.83 39.37 0)
+			(effects
+				(font
+					(size 1.27 1.27)
+				)
+				(hide yes)
+			)
+		)
+		(pin "2"
+		)
+		(pin "1"
+		)
+		(instances
+			(project ""
+				(path "/81126baf-9999-480c-992f-3520723c9b7d"
+					(reference "BT1")
+					(unit 1)
+				)
+			)
+		)
+	)
+	(symbol
+		(lib_id "power:GND")
+		(at 36.83 41.91 0)
+		(unit 1)
+		(exclude_from_sim no)
+		(in_bom yes)
+		(on_board yes)
+		(dnp no)
+		(fields_autoplaced yes)
+		(property "Reference" "#PWR02"
+			(at 36.83 48.26 0)
+			(effects
+				(font
+					(size 1.27 1.27)
+				)
+				(hide yes)
+			)
+		)
+		(property "Value" "GND"
+			(at 36.83 46.99 0)
+			(effects
+				(font
+					(size 1.27 1.27)
+				)
+			)
+		)
+		(property "Footprint" ""
+			(at 36.83 41.91 0)
+			(effects
+				(font
+					(size 1.27 1.27)
+				)
+				(hide yes)
+			)
+		)
+		(property "Datasheet" ""
+			(at 36.83 41.91 0)
+			(effects
+				(font
+					(size 1.27 1.27)
+				)
+				(hide yes)
+			)
+		)
+		(property "Description" "Power symbol creates a global label with name \"GND\" , ground"
+			(at 36.83 41.91 0)
+			(effects
+				(font
+					(size 1.27 1.27)
+				)
+				(hide yes)
+			)
+		)
+		(pin "1"
+		)
+		(instances
+			(project ""
+				(path "/81126baf-9999-480c-992f-3520723c9b7d"
+					(reference "#PWR02")
+					(unit 1)
+				)
+			)
+		)
+	)
 	(sheet_instances
 		(path "/"

Commit message: nothing new
Parts:
- added U1: ATtiny85-20M, Package_DFN_QFN:QFN-20-1EP_4x4mm_P0.5mm_EP2.6x2.6mm, symbol MCU_Microchip_ATtiny:ATtiny85-20M
Connections:
- net +3V0: now also U1.15 (VCC)
- net GND: now also U1.21 (GND), U1.8 (GND)
Changed lines of the file:
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@@
+	)
+	(symbol
+		(lib_id "power:GND")
+		(at 119.38 80.01 0)
+		(unit 1)
+		(exclude_from_sim no)
+		(in_bom yes)
+		(on_board yes)
+		(dnp no)
+		(fields_autoplaced yes)
+		(property "Reference" "#PWR04"
+			(at 119.38 86.36 0)
+			(effects
+				(font
+					(size 1.27 1.27)
+				)
+				(hide yes)
+			)
+		)
+		(property "Value" "GND"
+			(at 119.38 85.09 0)
+			(effects
+				(font
+					(size 1.27 1.27)
+				)
+			)
+		)
+		(property "Footprint" ""
+			(at 119.38 80.01 0)
+			(effects
+				(font
+					(size 1.27 1.27)
+				)
+				(hide yes)
+			)
+		)
+		(property "Datasheet" ""
+			(at 119.38 80.01 0)
+			(effects
+				(font
+					(size 1.27 1.27)
+				)
+				(hide yes)
+			)
+		)
+		(property "Description" "Power symbol creates a global label with name \"GND\" , ground"
+			(at 119.38 80.01 0)
+			(effects
+				(font
+					(size 1.27 1.27)
+				)
+				(hide yes)
+			)
+		)
+		(pin "1"
+		)
+		(instances
+			(project ""
+				(path "/81126baf-9999-480c-992f-3520723c9b7d"
+					(reference "#PWR04")
+					(unit 1)
+				)
+			)
+		)
 	)
 	(symbol
@@
 	)
 	(symbol
+		(lib_id "MCU_Microchip_ATtiny:ATtiny85-20M")
+		(at 119.38 64.77 0)
+		(unit 1)
+		(exclude_from_sim no)
+		(in_bom yes)
+		(on_board yes)
+		(dnp no)
+		(fields_autoplaced yes)
+		(property "Reference" "U1"
+			(at 105.41 63.4999 0)
+			(effects
+				(font
+					(size 1.27 1.27)
+				)
+				(justify right)
+			)
+		)
+		(property "Value" "ATtiny85-20M"
+			(at 105.41 66.0399 0)
+			(effects
+				(font
+					(size 1.27 1.27)
+				)
+				(justify right)
+			)
+		)
+		(property "Footprint" "Package_DFN_QFN:QFN-20-1EP_4x4mm_P0.5mm_EP2.6x2.6mm"
+			(at 119.38 64.77 0)
+			(effects
+				(font
+					(size 1.27 1.27)
+					(italic yes)
+				)
+				(hide yes)
+			)
+		)
+		(property "Datasheet" "http://ww1.microchip.com/downloads/en/DeviceDoc/atmel-2586-avr-8-bit-microcontroller-attiny25-attiny45-attiny85_datasheet.pdf"
+			(at 119.38 64.77 0)
+			(effects
+				(font
+					(size 1.27 1.27)
+				)
+				(hide yes)
+			)
+		)
+		(property "Description" "20MHz, 8kB Flash, 512B SRAM, 512B EEPROM, debugWIRE, QFN-20"
+			(at 119.38 64.77 0)
+			(effects
+				(font
+					(size 1.27 1.27)
+				)
+				(hide yes)
+			)
+		)
+		(pin "6"
+		)
+		(pin "4"
+		)
+		(pin "3"
+		)
+		(pin "7"
+		)
+		(pin "9"
+		)
+		(pin "10"
+		)
+		(pin "13"
+		)
+		(pin "20"
+		)
+		(pin "5"
+		)
+		(pin "16"
+		)
+		(pin "2"
+		)
+		(pin "12"
+		)
+		(pin "1"
+		)
+		(pin "18"
+		)
+		(pin "17"
+		)
+		(pin "8"
+		)
+		(pin "21"
+		)
+		(pin "11"
+		)
+		(pin "14"
+		)
+		(pin "19"
+		)
+		(pin "15"
+		)
+		(instances
+			(project ""
+				(path "/81126baf-9999-480c-992f-3520723c9b7d"
+					(reference "U1")
+					(unit 1)
+				)
+			)
+		)
+	)
+	(symbol
 		(lib_id "Device:Battery_Cell")
 		(at 36.83 39.37 0)
@@
 					(unit 1)
 				)
+			)
+		)
+	)
+	(symbol
+		(lib_id "power:+3V0")
+		(at 119.38 49.53 0)
+		(unit 1)
+		(exclude_from_sim no)
+		(in_bom yes)
+		(on_board yes)
+		(dnp no)
+		(fields_autoplaced yes)
+		(property "Reference" "#PWR03"
+			(at 119.38 53.34 0)
+			(effects
+				(font
+					(size 1.27 1.27)
+				)
+				(hide yes)
+			)
+		)
+		(property "Value" "+3V0"
+			(at 119.38 44.45 0)
+			(effects
+				(font
+					(size 1.27 1.27)
+				)
+			)
+		)
+		(property "Footprint" ""
+			(at 119.38 49.53 0)
+			(effects
+				(font
+					(size 1.27 1.27)
+				)
+				(hide yes)
+			)
+		)
+		(property "Datasheet" ""
+			(at 119.38 49.53 0)
+			(effects
+				(font
+					(size 1.27 1.27)
+				)
+				(hide yes)
+			)
+		)
+		(property "Description" "Power symbol creates a global label with name \"+3V0\""
+			(at 119.38 49.53 0)
+			(effects
+				(font
+					(size 1.27 1.27)
+				)
+				(hide yes)
+			)
+		)
+		(pin "1"
+		)
+		(instances
+			(project ""
+				(path "/81126baf-9999-480c-992f-3520723c9b7d"
+					(reference "#PWR03")
+					(unit 1)
+				)

Commit message: updated schematic
Parts:
- added BLUE_LED, LOST_LED, RED_LED, WON_LED, YELLOW_LED: LED, symbol Device:LED
- added BZ1: Buzzer, symbol Device:Buzzer
- added C1: 10uF, symbol Device:C
- added C2: 0.1uF, symbol Device:C
- added R1, R2, R3, R4, R5, R6, R7, R8: R_US, symbol Device:R_US
- added RESET, SW1, SW2, SW3: SW_Push, symbol Switch:SW_Push
Connections:
- net +3V0: now also C1.1, R4.1
- net GND: now also BZ1.2 (-), C1.2, C2.2, R5.1, R6.1, R7.1, R8.1
- new net: LOST_LED.2 (A), R1.2, RED_LED.1 (K), YELLOW_LED.2 (A)
- new net: BLUE_LED.1 (K), R2.2, RED_LED.2 (A), WON_LED.2 (A), YELLOW_LED.1 (K)
- new net: R7.2, SW3.1
- new net: R6.2, SW2.1
- new net: BLUE_LED.2 (A), LOST_LED.1 (K), R3.2, WON_LED.1 (K)
- new net: R5.2, SW1.1
- new net: R8.2, RESET.1
- new net 14: R1.1
- new net 15: R3.1
- new net 32: R2.1
- new net PB?: BZ1.1 (+), C2.1, R4.2, RESET.2, SW1.2, SW2.2, SW3.2
- no-connect marks 0 -> 1
Other:
- moved on the sheet: U1

Commit message: updated schematic
Parts:
- added R9: R_US, symbol Device:R_US
- R1, R2, R3: value R_US -> 220Ω
Connections:
- net 14 is gone; now on an unnamed net: R1.1
- net 15 is gone; now on net PB2: R3.1
- net 32 is gone; now on net PB1: R2.1
- net +3V0: now also R8.1
- net GND: now also R9.2; no longer R8.1
- net RESET: now reaches U1.1 (~{RESET}/PB5)
- net RESET: now also RESET.2, R9.1
- net at U1.11 (AREF/PB0): no longer names the net of U1.11 (AREF/PB0)
- net PB1: now reaches U1.12 (PB1)
- net PB2: now reaches U1.14 (PB2)
- net PB3: now reaches U1.2 (XTAL1/PB3)
- net PB3: now also C2.1, R4.2, SW1.2, SW2.2, SW3.2
- net PB5: now reaches U1.5 (XTAL2/PB4)
- net PB5: now also BZ1.1 (+)
- removed net PB?: BZ1.1 (+), C2.1, R4.2, RESET.2, SW1.2, SW2.2, SW3.2
Other:
- moved on the sheet: R1, R2, R3

Commit message: updated schemaatics
Parts:
- added J1: Conn_01x07, symbol Connector_Generic:Conn_01x07
- R8: value R_US -> 200Ω
Connections:
- net +3V0: now also J1.3 (Pin_3)
- net GND: now also J1.2 (Pin_2)
- net PB2: now also J1.5 (Pin_5)
- net at R1.1, U1.11 (AREF/PB0): now also J1.7 (Pin_7)
- net PB1 renamed MISO
- net MISO: now also J1.6 (Pin_6)
- net PB3 renamed CS
- net CS: now also J1.4 (Pin_4)
