File: Business_Card.kicad_sch (KiCad schematic)
At the start: 24 parts, among them J2 Conn_01x06, SW1 B3SN-3012P, SW2 B3SN-3012P, SW3 B3SN-3012P, U1 ATtiny85-20M

Commit message: Finished PCB
Parts:
- R1, R2, R3, R8, R9: footprint BUSINESS_CARD:R_0221 -> BUSINESS_CARD:221_R_RESC1005X40N
Connections:
- net +3V0: no longer J2.5 (Pin_5)
- no-connect marks 0 -> 1
Changed lines of the file:
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@@
 		(color 0 0 0 0)
+	)
+	(no_connect
+		(at 39.37 78.74)
 	)
 	(wire
@@
 			)
 		)
-		(property "Footprint" "BUSINESS_CARD:R_0221"
+		(property "Footprint" "BUSINESS_CARD:221_R_RESC1005X40N"
 			(at 112.776 51.054 90)
 			(effects
@@
 			)
 		)
-		(property "Footprint" "BUSINESS_CARD:R_0221"
+		(property "Footprint" "BUSINESS_CARD:221_R_RESC1005X40N"
 			(at 143.764 19.304 90)
 			(effects
@@
 	)
 	(symbol
-		(lib_id "power:+3V0")
-		(at 39.37 78.74 270)
-		(unit 1)
-		(exclude_from_sim no)
-		(in_bom yes)
-		(on_board yes)
-		(dnp no)
-		(fields_autoplaced yes)
-		(property "Reference" "#PWR013"
-			(at 35.56 78.74 0)
-			(effects
-				(font
-					(size 1.27 1.27)
-				)
-				(hide yes)
-			)
-		)
-		(property "Value" "+3V0"
-			(at 43.18 78.7399 90)
-			(effects
-				(font
-					(size 1.27 1.27)
-				)
-				(justify left)
-			)
-		)
-		(property "Footprint" ""
-			(at 39.37 78.74 0)
-			(effects
-				(font
-					(size 1.27 1.27)
-				)
-				(hide yes)
-			)
-		)
-		(property "Datasheet" ""
-			(at 39.37 78.74 0)
-			(effects
-				(font
-					(size 1.27 1.27)
-				)
-				(hide yes)
-			)
-		)
-		(property "Description" "Power symbol creates a global label with name \"+3V0\""
-			(at 39.37 78.74 0)
-			(effects
-				(font
-					(size 1.27 1.27)
-				)
-				(hide yes)
-			)
-		)
-		(pin "1"
-		)
-		(instances
-			(project ""
-				(path "/81126baf-9999-480c-992f-3520723c9b7d"
-					(reference "#PWR013")
-					(unit 1)
-				)
-			)
-		)
-	)
-	(symbol
 		(lib_id "Device:R_US")
 		(at 143.51 35.56 90)
@@
 			)
 		)
-		(property "Footprint" "BUSINESS_CARD:R_0221"
+		(property "Footprint" "BUSINESS_CARD:221_R_RESC1005X40N"
 			(at 143.764 34.544 90)
 			(effects
@@
 			)
 		)
-		(property "Footprint" "BUSINESS_CARD:R_0221"
+		(property "Footprint" "BUSINESS_CARD:221_R_RESC1005X40N"
 			(at 181.864 83.566 90)
 			(effects
@@
 			)
 		)
-		(property "Footprint" "BUSINESS_CARD:R_0221"
+		(property "Footprint" "BUSINESS_CARD:221_R_RESC1005X40N"
 			(at 143.764 26.924 90)
 			(effects
